File: pj4_MCU.kicad_pcb (KiCad board)
At the start: 4 copper layers, 54.4 x 38.1 mm, 29 parts, among them J1 Conn_01x09_Male, J2 Conn_02x03_Odd_Even, J3 Conn_01x04_Male, J4 Conn_01x04_Male, U1 24LC1025, U2 DS1337S+, U3 24LC1025, U4 ATMEGA328P-AU, Y1 32.768 KHz, Y2 16 MHz

Commit message: update MCU_PCB
Other:
- board text added: "- 2Mbits EEPRAM - RTC - I2C, SPI, GPIOs"
- board text added: "ICSP"
- board text removed: "- 2Mbits EEPRAM - RTC - I2C, SPI, GPIO"
Changed lines of the file:
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@@
       (drillshape 0)
       (scaleselection 1)
-      (outputdirectory "pj4_MCU_gerber/")
+      (outputdirectory "pj5_MCU_gerber_4_layer/")
     )
   )
@@
     (property "Sheetname" "")
     (attr smd)
-    (fp_text reference "U3" (at 0 -3.4) (layer "F.SilkS")
+    (fp_text reference "U3" (at 5.014 -1.966) (layer "F.SilkS")
       (effects (font (size 1 1) (thickness 0.15)))
     )
-    (fp_text value "24LC1025" (at 0 3.4) (layer "F.Fab")
+    (fp_text value "24LC1025" (at 0 3.4) (layer "F.SilkS")
       (effects (font (size 1 1) (thickness 0.15)))
     )
@@
       (effects (font (size 0.641239 0.641239) (thickness 0.15)))
     )
-    (fp_text value "ATMEGA328P-AU" (at 3.013915 6.107875) (layer "F.Fab")
+    (fp_text value "ATMEGA328P-AU" (at 3.013915 6.107875) (layer "F.SilkS")
       (effects (font (size 0.640449 0.640449) (thickness 0.15)))
     )
@@
     (property "Sheetname" "")
     (attr through_hole)
-    (fp_text reference "U2" (at -0.795 -3.332) (layer "F.SilkS")
+    (fp_text reference "U2" (at 5.014 -0.95) (layer "F.SilkS")
       (effects (font (size 1 1) (thickness 0.15)))
     )
@@
       (effects (font (size 1 1) (thickness 0.15)))
     )
-    (fp_text value "24LC1025" (at 0 3.4) (layer "F.Fab")
+    (fp_text value "24LC1025" (at 0 3.4) (layer "F.SilkS")
       (effects (font (size 1 1) (thickness 0.15)))
     )
@@
     (effects (font (size 1.5 1.5) (thickness 0.3)) (justify left mirror))
   )
-  (gr_text "- 2Mbits EEPRAM\n- RTC\n- I2C, SPI, GPIO\n" (at 145.354 130.998) (layer "B.SilkS")
+  (gr_text "- 2Mbits EEPRAM\n- RTC\n- I2C, SPI, GPIOs\n" (at 145.354 130.998) (layer "B.SilkS")
     (effects (font (size 1.5 1.5) (thickness 0.3)) (justify left mirror))
   )
@@
     (effects (font (size 1 1) (thickness 0.15)))
   )
+  (gr_text "ICSP" (at 155.448 121.412) (layer "F.SilkS")
+    (effects (font (size 1 1) (thickness 0.15)))
+  )
